Commit message: hybrid_cpp: replace URDFs with the official UR ROS2 description
A web survey of UR3e/UR10e inertial parameters turned up at least three
distinct sources, each with materially different mass/inertia values:

  • our previous URDFs   — CAD-derived, full inertia tensor
  • UR official ROS2     — UR-spec masses + cylindrical primitives
  • Robotics Toolbox UR  — masses only, no inertia

Most striking discrepancy: UR10e wrist_3 mass was 0.615 in our URDF
vs 0.202 in the UR official YAML — a 3× over-estimate that propagates
through Coriolis and gravity terms on the wrist. Several other links
also differed by 5–22% in mass and order-of-magnitude in inertia
elements.

Replace both URDFs with the UR official versions (sourced from the
Daniella1/urdf_files_dataset mirror of ros-industrial/ur_description,
generated from the UR-curated xacros). KDL chain (base_link → tool0)
remains identical so DynamicsModel/DOB/4CH stay wired exactly as
before — only the underlying inertial parameters change.

Self-test diff at home pose:

  UR10e M(q) diag old → new:
    [3.27, 7.33, 2.71, 0.046, 0.0083, 0.0003]
    [2.70, 6.72, 2.11, 0.044, 0.0073, 0.0002]   (most lighter, wrist_3 -33%)

  UR3e M(q) diag old → new:
    [0.276, 0.467, 0.191, 0.0107, 0.0021, 0.0001]
    [0.263, 0.417, 0.166, 0.0147, 0.0042, 0.0002] (wrists +37 to +100%)

The fundamental "lighter than passive" inequality KF > κ/M still
doesn't fit inside the stability bound KF < ~0.5/M, but with the new
URDF the model error inside the DOB residual should be smaller — so
cross-coupling at the round-2 KF=0.3 baseline may be lower, and the
stability margin at higher KF a little wider. Empirical question.

Round-2 baseline config kept (KP, KD, KF shared, κ=0.7).

Co-Authored-By: Claude Opus 4.7 (1M context) <noreply@anthropic.com>

File: ur10e_teleop_control_hybrid_cpp/resources/ur10e.urdf (robot description, URDF)
Before this commit: robot ur10, 13 links, 12 joints
Links:
- removed link ft_frame
- removed link world
- link forearm_link: mass 3.989 -> 3.87
- link shoulder_link: mass 7.369 -> 7.778
- link upper_arm_link: mass 13.051 -> 12.93
- link wrist_1_link: mass 2.1 -> 1.96
- link wrist_2_link: mass 1.98 -> 1.96
- link wrist_3_link: mass 0.615 -> 0.202
Joints:
- removed joint base_joint
- removed joint wrist_3_link-ft_frame
- joint wrist_1_joint: limit lower=-6.283185307179586 upper=6.283185307179586 effort=54.0 velocity=3.141592653589793 -> lower=-6.283185307179586 upper=6.283185307179586 effort=56.0 velocity=3.141592653589793
- joint wrist_2_joint: limit lower=-6.283185307179586 upper=6.283185307179586 effort=54.0 velocity=3.141592653589793 -> lower=-6.283185307179586 upper=6.283185307179586 effort=56.0 velocity=3.141592653589793
- joint wrist_3_joint: limit lower=-6.283185307179586 upper=6.283185307179586 effort=54.0 velocity=3.141592653589793 -> lower=-6.283185307179586 upper=6.283185307179586 effort=56.0 velocity=3.141592653589793

File: ur10e_teleop_control_hybrid_cpp/resources/ur3e.urdf (robot description, URDF)
Before this commit: robot ur3, 13 links, 12 joints
Links:
- removed link ft_frame
- removed link world
- link forearm_link: mass 1.437 -> 1.26
- link shoulder_link: mass 1.98 -> 2.0
- link upper_arm_link: mass 3.4445 -> 3.42
- link wrist_1_link: mass 0.871 -> 0.8
- link wrist_2_link: mass 0.805 -> 0.8
- link wrist_3_link: mass 0.261 -> 0.35
Joints:
- removed joint base_joint
- removed joint wrist_3_link-ft_frame
- joint shoulder_lift_joint: limit lower=-6.283185307179586 upper=6.283185307179586 effort=54.0 velocity=3.141592653589793 -> lower=-6.283185307179586 upper=6.283185307179586 effort=56.0 velocity=3.141592653589793
- joint shoulder_pan_joint: limit lower=-6.283185307179586 upper=6.283185307179586 effort=54.0 velocity=3.141592653589793 -> lower=-6.283185307179586 upper=6.283185307179586 effort=56.0 velocity=3.141592653589793
- joint wrist_1_joint: limit lower=-6.283185307179586 upper=6.283185307179586 effort=9.0 velocity=6.283185307179586 -> lower=-6.283185307179586 upper=6.283185307179586 effort=12.0 velocity=6.283185307179586
- joint wrist_2_joint: limit lower=-6.283185307179586 upper=6.283185307179586 effort=9.0 velocity=6.283185307179586 -> lower=-6.283185307179586 upper=6.283185307179586 effort=12.0 velocity=6.283185307179586
- joint wrist_3_joint: limit effort=9.0 velocity=6.283185307179586 -> lower=-6.283185307179586 upper=6.283185307179586 effort=12.0 velocity=6.283185307179586; type continuous -> revolute
