Commit message: oa_fd_cpp: fix joint1 axis in bundled URDF (z -> -y): j1 is a PITCH joint
HW evidence: q1=+1.49 tilts the arm back-horizontal and it free-falls when
released — joint1 is gravity-loaded pitch, not vertical yaw as the V10 URDF
claimed. Axis derived from measured poses (q2=-1.62 = left-horizontal fixes
y0=right; right-hand rule with q1=+1.49=back gives axis 0 -1 0). Verified:
prediction reproduces measured g[1]=-14.5 at the bent pose and adds
g[0]=+/-20.8 at fore/aft horizontal.

Co-Authored-By: Claude Opus 4.8 (1M context) <noreply@anthropic.com>

File: oa_fd_cpp/urdf/openarmx_arm.urdf (robot description, URDF)
Before this commit: robot openarmx, 10 links, 9 joints
Joints:
- joint openarmx_joint1: axis 0 0 1 -> 0 -1 0
