Commit message: fit_gravity.py: CRITICAL fix — joint k torque must sum DISTAL links only
The regressor summed ALL links 1-7 into every joint's torque equation.
Statics: only links distal to joint k load it; proximal links entered with
huge lever arms = phantom torques growing down the chain (verified against
the runtime-KDL tau_model column: j1-j3 ~0, j4 3.6, j6/j7 up to 11 Nm).

Fallout now explained:
- the 'j6/j7 telemetry broken, 7-8Nm' story was FALSE — measured j6/j7
  match runtime KDL at rms 0.2Nm; the 8Nm was the regressor's own phantom
- every previous fit URDF was poisoned (clamped COMs, wild masses), which
  is why none of them ever beat plain v2com on hardware
- --drop-joints 'helped' only because it dropped the corrupted equations

After the fix the offline regressor matches runtime KDL to 5e-5 Nm on all
7 joints. First clean fit (static, links 1-7, masses pinned):
mean 0.543 -> 0.279 Nm, max 4.74 -> 1.63 Nm, link4-7 COMs stay physical.
-> urdf/openarmx_arm_cali_left_leader.urdf regenerated (clean).
-> openarmx_arm_cali_combined.urdf deleted (poisoned-fit artifact).

Co-Authored-By: Claude Opus 4.8 (1M context) <noreply@anthropic.com>

File: oa_fd_cpp/urdf/openarmx_arm_cali_left_leader.urdf (robot description, URDF)
Before this commit: robot openarmx, 10 links, 9 joints
Links:
- link openarmx_link1: mass 1.141076 -> 1.141700
- link openarmx_link2: mass 0.276876 -> 0.277500
- link openarmx_link3: mass 1.073276 -> 1.073900
- link openarmx_link4: mass 0.634276 -> 0.634900
- link openarmx_link5: mass 0.615076 -> 0.615700
- link openarmx_link6: mass 0.474576 -> 0.475200
- link openarmx_link7: mass 0.624348 -> 0.624972
