Commit message: follower URDF rebuilt = leader arm (link0-6) + link7-only gripper fit
The full --fit-links 1-7 follower fit was DEGENERATE: links 2-5 COMs came out
unphysically different from the leader (q4/q5 COM-z even sign-flipped) though
it's the SAME arm — both fits hit residual 0.22 but landed in different
non-physical solutions, and the heavy gripper amplified the follower's into
the q1 horizontal-start runaway.

Physics says only the END TOOL differs, so: freeze link0-6 at the validated
leader values, fit ONLY link7 (gripper, mass 1.047) on the follower data.
Result: link0-6 identical to leader (<0.001), link7 = gripper. Consistent
per-arm models (same arm -> same params; only the tip differs). Residual
0.40 (vs leader 0.22) — higher because the arm isn't re-fit, but PHYSICAL.

HW-verify: follower-left should now stay put at the horizontal start like
the leader does (no q1 swing-back).

Co-Authored-By: Claude Opus 4.8 (1M context) <noreply@anthropic.com>

File: oa_fd_cpp/urdf/openarmx_arm_cali_left_follower.urdf (robot description, URDF)
Before this commit: robot openarmx, 10 links, 9 joints
Links:
- link openarmx_link2: mass 0.277500 -> 0.277484
- link openarmx_link3: mass 1.073900 -> 1.073864
- link openarmx_link4: mass 0.634900 -> 0.634836
- link openarmx_link5: mass 0.615700 -> 0.615599
- link openarmx_link6: mass 0.475200 -> 0.475059
- link openarmx_link7: mass 1.047023 -> 1.046883

File: oa_fd_cpp/urdf/openarmx_arm_cali_right_follower.urdf (robot description, URDF)
Before this commit: robot openarmx, 10 links, 9 joints
Links:
- link openarmx_link2: mass 0.277500 -> 0.277480
- link openarmx_link3: mass 1.073900 -> 1.073862
- link openarmx_link4: mass 0.634900 -> 0.634833
- link openarmx_link5: mass 0.615700 -> 0.615601
- link openarmx_link6: mass 0.475200 -> 0.475067
- link openarmx_link7: mass 1.047023 -> 1.046889

Commit message: revert follower URDFs to full-fit (a4a0dc1): link7-only made g1 HIGHER -> regressed follower-right q1
link7-only (leader arm + gripper) gave the HIGHEST horizontal g1 (+9.38 vs
full-fit +8.71 vs leader +8.32) -> both followers swung back on HW. The
full-fit at least had follower-right q1 stable. Reverting to it; the
follower q1 overcomp at the horizontal/straight startup is the real open
issue (40-pose fit is degenerate + heavy gripper amplifies). Investigate
before re-fitting again.

Co-Authored-By: Claude Opus 4.8 (1M context) <noreply@anthropic.com>

File: oa_fd_cpp/urdf/openarmx_arm_cali_left_follower.urdf (robot description, URDF)
Before this commit: robot openarmx, 10 links, 9 joints
Links:
- link openarmx_link2: mass 0.277484 -> 0.277500
- link openarmx_link3: mass 1.073864 -> 1.073900
- link openarmx_link4: mass 0.634836 -> 0.634900
- link openarmx_link5: mass 0.615599 -> 0.615700
- link openarmx_link6: mass 0.475059 -> 0.475200
- link openarmx_link7: mass 1.046883 -> 1.047023

File: oa_fd_cpp/urdf/openarmx_arm_cali_right_follower.urdf (robot description, URDF)
Before this commit: robot openarmx, 10 links, 9 joints
Links:
- link openarmx_link2: mass 0.277480 -> 0.277500
- link openarmx_link3: mass 1.073862 -> 1.073900
- link openarmx_link4: mass 0.634833 -> 0.634900
- link openarmx_link5: mass 0.615601 -> 0.615700
- link openarmx_link6: mass 0.475067 -> 0.475200
- link openarmx_link7: mass 1.046889 -> 1.047023

Commit message: follower gravity model = leader model (gripper contribution is negligible, data-proven)
Decisive data check: real gripper gravity contribution (follower_tau_meas -
leader_model) is within noise (j1 +0.05+-0.63, j4 +0.14+-0.27 Nm), and the
LEADER model explains the follower's measured data to 0.237 mean residual --
essentially the same as the follower's own fit (0.218). So the follower's
real gravity ~= the leader's; the gripper barely affects gravity.

The follower's own gripper-FIT model overcompensated: it injects spurious
torque when extrapolated to the operating region -> q1/q4 unstable-equilibrium
runaway. The validated leader model fits the follower data nearly as well AND
is stable. So: follower URDF = leader URDF (copy). follower g1(q1) now matches
the stable leader exactly.

This also answers the user: q4 coverage was NOT the cause (leader had the same
coverage and is stable); the cause was the degenerate gripper-fit overcomp.
No re-cali needed.

Co-Authored-By: Claude Opus 4.8 (1M context) <noreply@anthropic.com>

File: oa_fd_cpp/urdf/openarmx_arm_cali_left_follower.urdf (robot description, URDF)
Before this commit: robot openarmx, 10 links, 9 joints
Links:
- link openarmx_link7: mass 1.047023 -> 0.624972

File: oa_fd_cpp/urdf/openarmx_arm_cali_right_follower.urdf (robot description, URDF)
Before this commit: robot openarmx, 10 links, 9 joints
Links:
- link openarmx_link7: mass 1.047023 -> 0.624972
