Commit message: follower-right URDF: link7 end mass 1.5x leader (0.625 -> 0.9375)
Operator request: follower gripper end is ~1.5x the leader handle. Bump
link7 mass 0.624972 -> 0.937458 (x1.5), inertia scaled x1.5 too (no effect
on gravity FF), COM unchanged -> link7 gravity contribution scales x1.5.
follower-right only; leader-right and both left arms untouched. Departs
from D20 (follower URDF == leader) deliberately per operator.

Co-Authored-By: Claude Opus 4.8 (1M context) <noreply@anthropic.com>

File: oa_fd_cpp/urdf/openarmx_arm_cali_right_follower.urdf (robot description, URDF)
Before this commit: robot openarmx, 10 links, 9 joints
Links:
- link openarmx_link7: mass 0.624972 -> 0.937458

Commit message: follower-right URDF: link7 end mass 0.5x leader (1.5x gave overcomp)
0.937458 -> 0.312486 (0.5x of leader handle 0.624972), inertia x0.5,
COM unchanged. Operator: 1.5x overcompensated; probing 0.5x.

Co-Authored-By: Claude Opus 4.8 (1M context) <noreply@anthropic.com>

File: oa_fd_cpp/urdf/openarmx_arm_cali_right_follower.urdf (robot description, URDF)
Before this commit: robot openarmx, 10 links, 9 joints
Links:
- link openarmx_link7: mass 0.937458 -> 0.312486

Commit message: follower-right URDF: link7 end mass 1.1x leader (narrowing from 1.5/0.5)
0.312486 -> 0.687469 (1.1x of leader 0.624972), inertia x1.1, COM same.

Co-Authored-By: Claude Opus 4.8 (1M context) <noreply@anthropic.com>

File: oa_fd_cpp/urdf/openarmx_arm_cali_right_follower.urdf (robot description, URDF)
Before this commit: robot openarmx, 10 links, 9 joints
Links:
- link openarmx_link7: mass 0.312486 -> 0.687469
