Commit message: oa_viz: actually strip collision blocks (tags with attributes)
regex missed <collision name=...> -> RViz tried to load *_symp.stl collision
meshes that aren't bundled. Visual-only URDF now references only bundled .dae.

File: oa_viz/urdf/oa_bimanual.urdf (robot description, URDF)
Before this commit: robot openarmx, 22 links, 21 joints
Links:
- link openarmx_body_link0: geometry visual mesh filename=package://oa_viz/meshes/body/v10/visual/body_link0.dae scale=1.0 1.0 1.0
- link openarmx_left_link0: geometry visual mesh filename=package://oa_viz/meshes/arm/v10/visual/link0.dae scale=1.0 -1.0 1.0
- link openarmx_left_link1: geometry visual mesh filename=package://oa_viz/meshes/arm/v10/visual/link1.dae scale=1.0 -1.0 1.0
- link openarmx_left_link2: geometry visual mesh filename=package://oa_viz/meshes/arm/v10/visual/link2.dae scale=1.0 -1.0 1.0
- link openarmx_left_link3: geometry visual mesh filename=package://oa_viz/meshes/arm/v10/visual/link3.dae scale=1.0 -1.0 1.0
- link openarmx_left_link4: geometry visual mesh filename=package://oa_viz/meshes/arm/v10/visual/link4.dae scale=1.0 1.0 1.0
- link openarmx_left_link5: geometry visual mesh filename=package://oa_viz/meshes/arm/v10/visual/link5.dae scale=1.0 -1.0 1.0
- link openarmx_left_link6: geometry visual mesh filename=package://oa_viz/meshes/arm/v10/visual/link6.dae scale=1.0 -1.0 1.0
- link openarmx_left_link7: geometry visual mesh filename=package://oa_viz/meshes/arm/v10/visual/link7.dae scale=1.0 -1.0 1.0
- link openarmx_right_link0: geometry visual mesh filename=package://oa_viz/meshes/arm/v10/visual/link0.dae scale=1.0 1.0 1.0
- link openarmx_right_link1: geometry visual mesh filename=package://oa_viz/meshes/arm/v10/visual/link1.dae scale=1.0 1.0 1.0
- link openarmx_right_link2: geometry visual mesh filename=package://oa_viz/meshes/arm/v10/visual/link2.dae scale=1.0 1.0 1.0
- link openarmx_right_link3: geometry visual mesh filename=package://oa_viz/meshes/arm/v10/visual/link3.dae scale=1.0 1.0 1.0
- link openarmx_right_link4: geometry visual mesh filename=package://oa_viz/meshes/arm/v10/visual/link4.dae scale=1.0 1.0 1.0
- link openarmx_right_link5: geometry visual mesh filename=package://oa_viz/meshes/arm/v10/visual/link5.dae scale=1.0 1.0 1.0
- link openarmx_right_link6: geometry visual mesh filename=package://oa_viz/meshes/arm/v10/visual/link6.dae scale=1.0 1.0 1.0
- link openarmx_right_link7: geometry visual mesh filename=package://oa_viz/meshes/arm/v10/visual/link7.dae scale=1.0 1.0 1.0
